File: kicadelecload/kicadelecload.kicad_sch (KiCad schematic)
At the start: 28 parts, among them Q1 IRF540N, Q2 IRF540N, Q3 IRF540N, Q4 IRF540N, Q5 IRF540N, U1 ESP32-S2-DEVKITC-1, U2 LM358, U3 TL431D

Commit message: ajustement précision lecture shunt
Parts:
- added Q6: 2N7000, Package_TO_SOT_THT:TO-92_Inline, symbol Transistor_FET:2N7000
- added U4: LM358, symbol Amplifier_Operational:LM358
- added resistance10, resistance12, resistance17: 1k, symbol Device:R
- added resistance18: 100, symbol Device:R
- added resistance19: 5100k, symbol Device:R
- added resistance20: 100k, symbol Device:R
- PWMcapacitor2: value 10uF -> 1uF
- resistance8: value 3k -> 10k
- resistance9: value 2k -> 40k
Connections:
- net 3.3V_J1_2: now also resistance20.1
- net GND: now also Q6.1 (S)
- net GNG_J1_22: now also resistance12.1
- net Lecture Vshunt: now also U4.6 (-), U4.7
- net Vref: now also resistance10.1, resistance12.2; no longer U3.1 (K), U3.2 (A), U3.3 (A), U3.6 (A), U3.7 (A), resistance13.2
- net Vshunt: now also resistance19.1
- net at U2.6 (-), resistance8.2: now also resistance17.2
- net Mode faible courant: now reaches U1.J3_12 (GPIO36)
- net Mode faible courant: now also resistance18.1
- new net: Q6.3 (D), resistance17.1
- new net: U3.1 (K), U3.2 (A), U3.3 (A), U3.6 (A), U3.7 (A), resistance10.2, resistance13.2
- new net: Q6.2 (G), resistance18.2
- new net: U4.5 (+), resistance19.2, resistance20.2
- no-connect marks 1 -> 0
Other:
- moved on the sheet: DS1, PWMcapacitor2, U2C, resistance16
