File: kicadelecload/_autosave-kicadelecload.kicad_sch (KiCad schematic)
At the start: 28 parts, among them Q1 IRF540N, Q2 IRF540N, Q3 IRF540N, Q4 IRF540N, Q5 IRF540N, U1 ESP32-S2-DEVKITC-1, U2 LM358, U3 TL431D

Commit message: adc adjustement and new pwm class
Parts:
- PWMcapacitor2: value 10uF -> 1uF
Changed lines of the file:
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@@
 			)
 		)
-		(property "Value" "10uF"
+		(property "Value" "1uF"
 			(at 114.554 118.11 90)
 			(effects
